File: schema_pcb/SupplyCircuit.sch (KiCad schematic (older format))
At the start: 26 parts, among them K1 Supply, U1 7805, U10 MC33063AD, U9 L7812

Commit message: update
Parts:
- L1: value 1m -> 470uH
Changed lines of the file:
@@
 P 3450 5850
 F 0 "L1" H 3503 5896 50  0000 L CNN
-F 1 "1m" H 3503 5805 50  0000 L CNN
+F 1 "470uH" H 3503 5805 50  0000 L CNN
 F 2 "Inductor_SMD:L_Bourns-SRR1005" H 3450 5850 50  0001 C CNN
 F 3 "~" H 3450 5850 50  0001 C CNN
